File: Battery.kicad_sch (KiCad schematic)
At the start: 25 parts, among them J1 USB, J2 USB_C_Receptacle_PowerOnly_6P, J3 BAT, Q1 SI2312BDS, Q2 SI2301BDS, U1 ME2801, U2 TP4056-42-ESOP8

Commit message: Schematic and board layout
Updated the project schematic.
Updated the board layout.
Parts:
- added R1: 10K, Resistor_SMD:R_0805_2012Metric, symbol Device:R
- D1: renamed from D2; value FULL -> STBY
- Q1, Q2, U1: footprint Package_TO_SOT_SMD:SOT-23 -> Custom_Parts:SOT-23_NO_MARK
- renumbered D1 to D2, R4 to R2, R1 to R4, R2 to R5, R5 to R6, R6 to R7, R7 to R8
Connections:
- net GBAT: now also Q1.2 (S); no longer Q1.3 (D)
- net GND: now also Q1.3 (D); no longer D1.1 (K), D2.1 (K), Q1.2 (S)
- net VUSB: now also D1.2 (A), D2.2 (A)
- net at R2.1: now also U2.6 (~{STDBY}); no longer D1.2 (A)
- net at R2.2: now also D1.1 (K); no longer U2.6 (~{STDBY})
- net at Q1.1 (G): now also R1.2; no longer U1.1 (SET)
- net at R3.1: now also U2.7 (~{CHRG}); no longer D2.2 (A)
- net at R3.2: now also D2.1 (K); no longer U2.7 (~{CHRG})
- new net: R1.1, U1.1 (SET)
Other:
- moved on the sheet: C1, C3, D1, D2, J3, R2, R3, R6, TP2, U1, U2
