File: Regulator.kicad_sch (KiCad schematic)
At the start: 19 parts, among them J4 OUT, U3 TLV61048DBVR, U4 TLV76701DRVx

Commit message: Schematic and board layout
Updated the project schematic.
Updated the board layout.
Parts:
- R10: renamed from R9; value 120K -> 10K
- R11: renamed from R10; value 10K -> 102K
- R12: renamed from R11; value 102K -> 10K
- R9: renamed from R8; value 10K -> 120K
Changed lines of the file:
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@@
 		(title "BATTERY MODULE")
 		(date "2025-03-27")
-		(rev "1.1")
+		(rev "1.2")
 		(company "Chapuzas S.L.")
 	)
@@
 		(on_board yes)
 		(dnp no)
-		(property "Reference" "R11"
+		(property "Reference" "R12"
 			(at 129.54 125.73 0)
 			(effects
@@
 			)
 		)
-		(property "Value" "102K"
-			(at 128.27 128.27 0)
+		(property "Value" "10K"
+			(at 129.54 128.27 0)
 			(effects
 				(font
@@
 			(project "BatteryModule"
 				(path "/31b6c323-c569-49bb-be2a-0e0809977ca4/860ba1b3-15a5-41eb-845b-167d81e21ddf"
-					(reference "R11")
+					(reference "R12")
 					(unit 1)
 				)
@@
 		(dnp no)
 		(fields_autoplaced yes)
-		(property "Reference" "#PWR037"
+		(property "Reference" "#PWR036"
 			(at 119.38 139.7 0)
 			(effects
@@
 			(project "BatteryModule"
 				(path "/31b6c323-c569-49bb-be2a-0e0809977ca4/860ba1b3-15a5-41eb-845b-167d81e21ddf"
-					(reference "#PWR037")
+					(reference "#PWR036")
 					(unit 1)
 				)
@@
 		(dnp no)
 		(fields_autoplaced yes)
-		(property "Reference" "#PWR027"
+		(property "Reference" "#PWR025"
 			(at 152.4 57.15 0)
 			(effects
@@
 			(project "BatteryModule"
 				(path "/31b6c323-c569-49bb-be2a-0e0809977ca4/860ba1b3-15a5-41eb-845b-167d81e21ddf"
-					(reference "#PWR027")
+					(reference "#PWR025")
 					(unit 1)
 				)
@@
 		(dnp no)
 		(fields_autoplaced yes)
-		(property "Reference" "#PWR032"
+		(property "Reference" "#PWR030"
 			(at 167.64 80.01 0)
 			(effects
@@
 			(project "BatteryModule"
 				(path "/31b6c323-c569-49bb-be2a-0e0809977ca4/860ba1b3-15a5-41eb-845b-167d81e21ddf"
-					(reference "#PWR032")
+					(reference "#PWR030")
 					(unit 1)
 				)
@@
 		(on_board yes)
 		(dnp no)
-		(property "Reference" "R8"
+		(property "Reference" "R9"
 			(at 149.86 60.96 90)
 			(effects
@@
 			)
 		)
-		(property "Value" "10K"
+		(property "Value" "120K"
 			(at 149.86 63.5 90)
 			(effects
@@
 			(project "BatteryModule"
 				(path "/31b6c323-c569-49bb-be2a-0e0809977ca4/860ba1b3-15a5-41eb-845b-167d81e21ddf"
-					(reference "R8")
+					(reference "R9")
 					(unit 1)
 				)
@@
 		(dnp no)
 		(fields_autoplaced yes)
-		(property "Reference" "#PWR033"
+		(property "Reference" "#PWR031"
 			(at 180.34 80.01 0)
 			(effects
@@
 			(project "BatteryModule"
 				(path "/31b6c323-c569-49bb-be2a-0e0809977ca4/860ba1b3-15a5-41eb-845b-167d81e21ddf"
-					(reference "#PWR033")
+					(reference "#PWR031")
 					(unit 1)
 				)
@@
 		(dnp no)
 		(fields_autoplaced yes)
-		(property "Reference" "#PWR044"
+		(property "Reference" "#PWR034"
 			(at 175.26 115.57 0)
 			(effects
@@
 			(project "BatteryModule"
 				(path "/31b6c323-c569-49bb-be2a-0e0809977ca4/860ba1b3-15a5-41eb-845b-167d81e21ddf"
-					(reference "#PWR044")
+					(reference "#PWR034")
 					(unit 1)
 				)
@@
 		(dnp no)
 		(fields_autoplaced yes)
-		(property "Reference" "#PWR030"
+		(property "Reference" "#PWR028"
 			(at 128.27 80.01 0)
 			(effects
@@
 			(project "BatteryModule"
 				(path "/31b6c323-c569-49bb-be2a-0e0809977ca4/860ba1b3-15a5-41eb-845b-167d81e21ddf"
-					(reference "#PWR030")
+					(reference "#PWR028")
 					(unit 1)
 				)
@@
 		(dnp no)
 		(fields_autoplaced yes)
-		(property "Reference" "#PWR031"
+		(property "Reference" "#PWR029"
 			(at 143.51 80.01 0)
 			(effects
@@
 			(project "BatteryModule"
 				(path "/31b6c323-c569-49bb-be2a-0e0809977ca4/860ba1b3-15a5-41eb-845b-167d81e21ddf"
-					(reference "#PWR031")
+					(reference "#PWR029")
 					(unit 1)
 				)
@@
 		(dnp no)
 		(fields_autoplaced yes)
-		(property "Reference" "#PWR035"
+		(property "Reference" "#PWR033"
 			(at 107.95 113.03 0)
 			(effects
@@
 			(project "BatteryModule"
 				(path "/31b6c323-c569-49bb-be2a-0e0809977ca4/860ba1b3-15a5-41eb-845b-167d81e21ddf"
-					(reference "#PWR035")
+					(reference "#PWR033")
 					(unit 1)
 				)
@@
 		(dnp no)
 		(fields_autoplaced yes)
-		(property "Reference" "#PWR040"
+		(property "Reference" "#PWR039"
 			(at 163.83 139.7 0)
 			(effects
@@
 			(project "BatteryModule"
 				(path "/31b6c323-c569-49bb-be2a-0e0809977ca4/860ba1b3-15a5-41eb-845b-167d81e21ddf"
-					(reference "#PWR040")
+					(reference "#PWR039")
 					(unit 1)
 				)
@@
 		(dnp no)
 		(fields_autoplaced yes)
-		(property "Reference" "#PWR025"
+		(property "Reference" "#PWR023"
 			(at 106.68 52.07 0)
 			(effects
@@
 			(project "BatteryModule"
 				(path "/31b6c323-c569-49bb-be2a-0e0809977ca4/860ba1b3-15a5-41eb-845b-167d81e21ddf"
-					(reference "#PWR025")
+					(reference "#PWR023")
 					(unit 1)
 				)
@@
 		(dnp no)
 		(fields_autoplaced yes)
-		(property "Reference" "#PWR039"
+		(property "Reference" "#PWR038"
 			(at 153.67 139.7 0)
 			(effects
@@
 			(project "BatteryModule"
 				(path "/31b6c323-c569-49bb-be2a-0e0809977ca4/860ba1b3-15a5-41eb-845b-167d81e21ddf"
-					(reference "#PWR039")
+					(reference "#PWR038")
 					(unit 1)
 				)
@@
 		(dnp no)
 		(fields_autoplaced yes)
-		(property "Reference" "#PWR038"
+		(property "Reference" "#PWR037"
 			(at 135.89 139.7 0)
 			(effects
@@
 			(project "BatteryModule"
 				(path "/31b6c323-c569-49bb-be2a-0e0809977ca4/860ba1b3-15a5-41eb-845b-167d81e21ddf"
-					(reference "#PWR038")
+					(reference "#PWR037")
 					(unit 1)
 				)
@@
 		(dnp no)
 		(fields_autoplaced yes)
-		(property "Reference" "#PWR036"
+		(property "Reference" "#PWR035"
 			(at 106.68 139.7 0)
 			(effects
@@
 			(project "BatteryModule"
 				(path "/31b6c323-c569-49bb-be2a-0e0809977ca4/860ba1b3-15a5-41eb-845b-167d81e21ddf"
-					(reference "#PWR036")
+					(reference "#PWR035")
 					(unit 1)
 				)
@@
 		(dnp no)
 		(fields_autoplaced yes)
-		(property "Reference" "R10"
+		(property "Reference" "R11"
 			(at 142.24 109.22 90)
 			(effects
@@
 			)
 		)
-		(property "Value" "10K"
+		(property "Value" "102K"
 			(at 142.24 111.76 90)
 			(effects
@@
 			(project "BatteryModule"
 				(path "/31b6c323-c569-49bb-be2a-0e0809977ca4/860ba1b3-15a5-41eb-845b-167d81e21ddf"
-					(reference "R10")
+					(reference "R11")
 					(unit 1)
 				)
@@
 		(dnp no)
 		(fields_autoplaced yes)
-		(property "Reference" "#PWR034"
+		(property "Reference" "#PWR032"
 			(at 148.59 114.3 0)
 			(effects
@@
 			(project "BatteryModule"
 				(path "/31b6c323-c569-49bb-be2a-0e0809977ca4/860ba1b3-15a5-41eb-845b-167d81e21ddf"
-					(reference "#PWR034")
+					(reference "#PWR032")
 					(unit 1)
 				)
@@
 		(on_board yes)
 		(dnp no)
-		(property "Reference" "R9"
+		(property "Reference" "R10"
 			(at 137.16 62.23 0)
 			(effects
@@
 			)
 		)
-		(property "Value" "120K"
-			(at 135.89 64.77 0)
+		(property "Value" "10K"
+			(at 137.16 64.77 0)
 			(effects
 				(font
@@
 			(project "BatteryModule"
 				(path "/31b6c323-c569-49bb-be2a-0e0809977ca4/860ba1b3-15a5-41eb-845b-167d81e21ddf"
-					(reference "R9")
+					(reference "R10")
 					(unit 1)
 				)
@@
 		(dnp no)
 		(fields_autoplaced yes)
-		(property "Reference" "#PWR041"
+		(property "Reference" "#PWR040"
 			(at 179.07 139.7 0)
 			(effects
@@
 			(project "BatteryModule"
 				(path "/31b6c323-c569-49bb-be2a-0e0809977ca4/860ba1b3-15a5-41eb-845b-167d81e21ddf"
-					(reference "#PWR041")
+					(reference "#PWR040")
 					(unit 1)
 				)
@@
 		(dnp no)
 		(fields_autoplaced yes)
-		(property "Reference" "#PWR028"
+		(property "Reference" "#PWR026"
 			(at 105.41 80.01 0)
 			(effects
@@
 			(project "BatteryModule"
 				(path "/31b6c323-c569-49bb-be2a-0e0809977ca4/860ba1b3-15a5-41eb-845b-167d81e21ddf"
-					(reference "#PWR028")
+					(reference "#PWR026")
 					(unit 1)
 				)
@@
 		(dnp no)
 		(fields_autoplaced yes)
-		(property "Reference" "#PWR026"
+		(property "Reference" "#PWR024"
 			(at 179.07 52.07 0)
 			(effects
@@
 			(project "BatteryModule"
 				(path "/31b6c323-c569-49bb-be2a-0e0809977ca4/860ba1b3-15a5-41eb-845b-167d81e21ddf"
-					(reference "#PWR026")
+					(reference "#PWR024")
 					(unit 1)
 				)
@@
 		(dnp no)
 		(fields_autoplaced yes)
-		(property "Reference" "#PWR029"
+		(property "Reference" "#PWR027"
 			(at 118.11 80.01 0)
 			(effects
@@
 			(project "BatteryModule"
 				(path "/31b6c323-c569-49bb-be2a-0e0809977ca4/860ba1b3-15a5-41eb-845b-167d81e21ddf"
-					(reference "#PWR029")
+					(reference "#PWR027")
 					(unit 1)
 				)
